Commit message: second commit

File: src/kr20_kr120_description/urdf/kr20_kr120.urdf.xacro (robot description, xacro)
@@ -192,4 +192,15 @@
         <state_interface name="velocity"/>
       </joint>
+      <!-- KR120 gyro joints (so ros2_control exposes them) -->
+      <joint name="kr120_gyro_left_joint">
+        <command_interface name="velocity"/>
+        <state_interface   name="position"/>
+        <state_interface   name="velocity"/>
+      </joint>
+      <joint name="kr120_gyro_right_joint">
+        <command_interface name="velocity"/>
+        <state_interface   name="position"/>
+        <state_interface   name="velocity"/>
+      </joint>
     </ros2_control>
     <!--  pareti -->
